File: hardware/KiCad/wiring_diagram/wiring_diagram.kicad_sch (KiCad schematic)
At the start: 4 parts, among them U1 ESP32-WROOM-32, U2 MAX31865xAP

Commit message: update
Parts:
- added U3: LM2596S-3.3, Package_TO_SOT_SMD:TO-263-5_TabPin3, symbol Regulator_Switching:LM2596S-3.3
- R1: value R -> 430 Ω
Connections:
- net GND: now reaches U2.13 (GND), U2.19 (GND)
- net GND: now also U1.1 (GND), U1.15 (GND), U1.38 (GND), U1.39 (GND), U3.3 (GND)
- net at U2.14 (SDI): now also U1.37 (IO23)
- net at U2.15 (SCLK): now also U1.30 (IO18)
- net at U2.16 (~{CS}): now also U1.29 (IO5)
- net at U2.17 (SDO): now also U1.31 (IO19)
- net at U2.3 (VDD): now also U1.2 (VDD), U3.2 (OUT)
- new net +12V: U3.1 (VIN), U3.5 (~{ON}/OFF)
