File: KiCad/chargriller-980.kicad_sch (KiCad schematic)
At the start: 14 parts, among them J1 MAX31855, J2 Conn_01x04, J3 TM1637, J4 TM1637, M1 Fan_3pin, Q1 IRLZ44N, U1 ESP32-DEVKITC-32D, U2 INA219, U3 KY-040, U5 LM2596S-ADJ

Commit message: updates to KiCad files
Parts:
- removed J2: Conn_01x04, symbol Connector_Generic:Conn_01x04
- added SW1, SW2: SW_Push, symbol Switch:SW_Push
Connections:
- net +12V: now also D1.1 (K), M1.2 (+), U2.6 (VIN+), U2.VIN+, U5.1 (IN+)
- net GND: now also U2.5 (VIN-), U2.VIN-, U5.5 (IN-)
- net at J4.1 (CLK): now also U1.J3-2 (IO23)
- net at J4.2 (DIO): now also U1.J2-10 (IO26)
- net at J4.3 (VCC): now also J3.3 (VCC), U1.J2-19 (EXT_5V), U5.4 (OUT+)
- net at J4.4 (GND): now also BZ1.2 (-), J3.4 (GND), U5.2 (OUT-)
- net at U3.CLK: now also U1.J2-7 (IO32)
- net at U3.DT: now also U1.J2-8 (IO33)
- net at U3.GND: now also J1.1 (GND), U1.J3-1 (GND3), SW1.2
- net at U3.SW: now also U1.J2-11 (IO27)
- net at Q1.2 (D): now also R1.1
- net at Q1.3 (S): now also D1.2 (A), M1.1 (-)
- net at U1.J2-1 (3V3): now also J1.2 (VCC), U2.1 (VCC)
- net at U1.J2-12 (IO14): now also J1.4 (CS)
- net at U1.J2-15 (IO13): now also SW2.1
- net at U1.J2-9 (IO25): now also J3.1 (CLK)
- net at U1.J3-11 (IO17): now also U2.3 (SCL)
- net at U1.J3-12 (IO16): now also R1.2
- net at U1.J3-13 (IO4): now also BZ1.1 (+)
- net at U1.J3-3 (IO22): now also J3.2 (DIO)
- net at U1.J3-6 (IO21): now also U2.4 (SDA)
- net at U1.J3-8 (IO19): now also J1.3 (DO)
- net at U1.J3-9 (IO18): now also J1.5 (CLK)
- net at TC1.1 (+): now also J1.7 (YELLOW_+)
- net at TC1.2 (-): now also J1.6 (RED_-)
- new net: SW1.1, SW2.2
Other:
- moved on the sheet: BZ1, D1, J3, J4, M1, Q1, R1, U2, U3, U5

Commit message: further updates to KiCad schematic and remove auto_saved_files
Connections:
- net +12V: no longer D1.1 (K)
- net GND: now also Q1.3 (S)
- net at Q1.1 (G): now also R1.1
- net at Q1.2 (D): now also M1.1 (-); no longer R1.1
- now unconnected: D1.2 (A)
Other:
- moved on the sheet: Q1

Commit message: updates to KiCad schematic and gitignore
Parts:
- added R2: 10kΩ, symbol Device:R
- R1: value R -> 220Ω
Connections:
- net +12V: now also D1.1 (K)
- net GND: now also R2.1
- net at Q1.1 (G), R1.1: now also M1.3 (Tacho), R2.2
- net at M1.1 (-), Q1.2 (D): now also D1.2 (A)
Other:
- moved on the sheet: D1, M1, Q1

Commit message: feat: update KiCad files based on user changes
Parts:
- removed Q1: IRLZ44N, Package_TO_SOT_THT:TO-220-3_Vertical, symbol Transistor_FET:IRLZ44N
- added Q2: IRLZ34N, Package_TO_SOT_THT:TO-220-3_Vertical, symbol Transistor_FET:IRLZ34N
Connections:
- net GND: now also Q2.3 (S)
- net at J1.1 (GND), SW1.2, U1.J3-1 (GND3)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: now also R1.2, U1.J3-12 (IO16)
- net at M1.3 (Tacho), R1.1, R2.2: now also Q2.1 (G)
- net at D1.2 (A), M1.1 (-): now also Q2.2 (D)
Other:
- moved on the sheet: R1
